Commit message: Fix drone model: - Fixed drone weight, it is more lighter; - Added gaussian noise to sonar; - Minor fix to other sensors.
Signed-off-by: m-paini <m.paini@reply.it>

File: cvg_sim_gazebo/urdf/quadrotor.urdf.xacro (robot description, xacro)
@@ -1,11 +1,10 @@
 <?xml version="1.0"?>
-<robot name="quadrotor"
-    xmlns:sensor="http://playerstage.sourceforge.net/gazebo/xmlschema/#sensor"
-    xmlns:controller="http://playerstage.sourceforge.net/gazebo/xmlschema/#controller"
-    xmlns:interface="http://playerstage.sourceforge.net/gazebo/xmlschema/#interface"
-    xmlns:xacro="http://playerstage.sourceforge.net/gazebo/xmlschema/#interface">
+<robot
+  name="quadrotor"
+  xmlns:xacro="http://ros.org/wiki/xacro"
+>
     <!-- Included URDF Files -->
     <xacro:include filename="$(find cvg_sim_gazebo)/urdf/quadrotor_base.urdf.xacro" />
     <!-- Instantiate quadrotor_base_macro once (has no parameters atm) -->
-    <quadrotor_base_macro />
+    <xacro:quadrotor_base_macro />
 </robot>

File: cvg_sim_gazebo/urdf/quadrotor_base.urdf.xacro (robot description, xacro)
@@ -1,15 +1,11 @@
 <?xml version="1.0"?>
-<robot xmlns:sensor="http://playerstage.sourceforge.net/gazebo/xmlschema/#sensor"
-xmlns:controller="http://playerstage.sourceforge.net/gazebo/xmlschema/#controller"
-xmlns:interface="http://playerstage.sourceforge.net/gazebo/xmlschema/#interface"
-xmlns:xacro="http://ros.org/wiki/xacro"
->
+<robot xmlns:xacro="http://ros.org/wiki/xacro">
   <xacro:include filename="$(find cvg_sim_gazebo_plugins)/urdf/quadrotor_plugins.urdf.xacro" />
-  <property name="pi" value="3.1415926535897931" />
+  <xacro:property name="pi" value="3.1415926535897931" />
   <!-- Main quadrotor link -->
   <xacro:macro name="quadrotor_base_macro">
     <link name="base_link">
       <inertial>
-        <mass value="1.477" />
+        <mass value="0.420" />
         <origin xyz="0 0 0" />
         <inertia ixx="0.01152" ixy="0.0" ixz="0.0" iyy="0.01152" iyz="0.0" izz="0.0218" />

File: cvg_sim_gazebo/urdf/sensors/generic_camera.urdf.xacro (robot description, xacro)
@@ -1,37 +1,33 @@
 <?xml version="1.0"?>
-<robot xmlns:sensor="http://playerstage.sourceforge.net/gazebo/xmlschema/#sensor"
-xmlns:controller="http://playerstage.sourceforge.net/gazebo/xmlschema/#controller"
-xmlns:interface="http://playerstage.sourceforge.net/gazebo/xmlschema/#interface"
-  xmlns:xacro="http://ros.org/wiki/xacro"
-  >
-    <property name="M_PI" value="3.1415926535897931" />
-    <xacro:macro name="generic_camera" params="name sim_name parent *origin update_rate res_x res_y image_format hfov">
-      <joint name="${name}_joint" type="fixed">
-        <insert_block name="origin" />
-        <parent link="${parent}"/>
-        <child link="${name}_link"/>
-      </joint>
-      <link name="${name}_link">
-        <inertial>
-          <mass value="0.001" />
-          <origin xyz="0 0 0" rpy="0 0 0" />
-          <inertia ixx="0.0001" ixy="0" ixz="0" iyy="0.0001" iyz="0" izz="0.0001" />
-        </inertial>
-        <visual>
-          <origin xyz="0 0 0" rpy="0 0 0" />
-          <geometry>
-            <box size="0.01 0.01 0.01" />
-          </geometry>
-	  <material name="Blue">
-      <color rgba="0.0 0.0 0.8 1"/>
-    </material>
-        </visual>
-        <collision>
-          <origin xyz="0 0 0" rpy="0 0 0" />
-          <geometry>
-            <box size="0.01 0.01 0.01" />
-          </geometry>
-        </collision>
-      </link>
+<robot xmlns:xacro="http://ros.org/wiki/xacro">
+  <xacro:property name="M_PI" value="3.1415926535897931" />
+  <xacro:macro name="generic_camera" params="name sim_name parent *origin update_rate res_x res_y image_format hfov">
+    <joint name="${name}_joint" type="fixed">
+      <xacro:insert_block name="origin" />
+      <parent link="${parent}"/>
+      <child link="${name}_link"/>
+    </joint>
+    <link name="${name}_link">
+<!--      <inertial>
+        <mass value="0.001" />
+        <origin xyz="0 0 0" rpy="0 0 0" />
+        <inertia ixx="0.0001" ixy="0" ixz="0" iyy="0.0001" iyz="0" izz="0.0001" />
+      </inertial>
+      <visual>
+        <origin xyz="0 0 0" rpy="0 0 0" />
+        <geometry>
+          <box size="0.01 0.01 0.01" />
+        </geometry>
+        <material name="Blue">
+          <color rgba="0.0 0.0 0.8 1"/>
+        </material>
+      </visual>
+      <collision>
+        <origin xyz="0 0 0" rpy="0 0 0" />
+        <geometry>
+          <box size="0.01 0.01 0.01" />
+        </geometry>
+      </collision>-->
+    </link>
     <joint name="${name}_optical_joint" type="fixed">
       <origin xyz="0 0 0" rpy="${-M_PI/2} 0.0 ${-M_PI/2}" />
@@ -39,29 +35,9 @@
       <child link="ardrone_base_${name}cam"/>
     </joint>
-    <link name="ardrone_base_${name}cam">
-      <inertial>
-        <mass value="0.01" />
-        <origin xyz="0 0 0" />
-        <inertia ixx="0.001"  ixy="0.0"  ixz="0.0"
-                 iyy="0.001"  iyz="0.0"
-                 izz="0.001" />
-      </inertial>
-      <visual>
-        <origin xyz="0 0 0" rpy="0 0 0"/>
-        <geometry>
-          <box size="0.001 0.001 0.001" />
-        </geometry>
-      </visual>
-      <collision>
-        <origin xyz="0 0 0" rpy="0 0 0"/>
-        <geometry>
-          <box size="0.001 0.001 0.001" />
-        </geometry>
-      </collision>
-    </link>
+    <link name="ardrone_base_${name}cam"/>
     <gazebo reference="${name}_link">
       <sensor type="camera" name="${name}_camera_sensor">
         <update_rate>${update_rate}</update_rate>
-        <camera name="head">
+        <camera>
           <horizontal_fov>${hfov}</horizontal_fov>
           <image>
@@ -70,6 +46,6 @@
             <format>${image_format}</format>
           </image>
-          <clip>0.01
-	    <near>0.01</near>
+          <clip>
+	        <near>0.01</near>
             <far>100</far>
           </clip>
@@ -84,7 +60,5 @@
         </plugin>
       </sensor>
-      <turnGravityOff>true</turnGravityOff>
-      <material>Gazebo/Blue</material>
     </gazebo>
-    </xacro:macro>
-  </robot>
+   </xacro:macro>
+</robot>

File: cvg_sim_gazebo/urdf/sensors/sonar_sensor.urdf.xacro (robot description, xacro)
@@ -1,8 +1,4 @@
 <?xml version="1.0"?>
-<robot xmlns:sensor="http://playerstage.sourceforge.net/gazebo/xmlschema/#sensor"
-xmlns:controller="http://playerstage.sourceforge.net/gazebo/xmlschema/#controller"
-xmlns:interface="http://playerstage.sourceforge.net/gazebo/xmlschema/#interface"
-xmlns:xacro="http://ros.org/wiki/xacro"
->
+<robot xmlns:xacro="http://ros.org/wiki/xacro">
   <xacro:macro name="sonar_sensor" params="name parent *origin ros_topic update_rate min_range max_range field_of_view ray_count">
     <joint name="${name}_joint" type="fixed">
@@ -21,5 +17,5 @@
         <geometry>
           <!--<box size="0.01 0.01 0.01" /> -->
-          <mesh filename="package://cvg_sim_gazebo/meshes/sonar_sensor/max_sonar_ez4.dae"/>
+          <mesh filename="package://hector_sensors_description/meshes/sonar_sensor/max_sonar_ez4.dae"/>
         </geometry>
       </visual>
@@ -33,5 +29,8 @@
     <gazebo reference="${name}_link">
       <sensor type="ray" name="${name}">
+        <always_on>true</always_on>
         <update_rate>${update_rate}</update_rate>
+        <pose>0 0 0 0 0 0</pose>
+        <visualize>false</visualize>
         <ray>
           <range>
@@ -43,4 +42,5 @@
             <horizontal>
               <samples>${ray_count}</samples>
+              <resolution>1</resolution>
               <min_angle>-${field_of_view/2}</min_angle>
               <max_angle>${field_of_view/2}</max_angle>
@@ -54,5 +54,5 @@
         </ray>
         <plugin name="gazebo_ros_${name}_controller" filename="libhector_gazebo_ros_sonar.so">
-          <gaussianNoise>0.000</gaussianNoise>
+          <gaussianNoise>0.005</gaussianNoise>
           <topicName>${ros_topic}</topicName>
           <frameId>${name}_link</frameId>

File: cvg_sim_gazebo_plugins/urdf/quadrotor_sensors.urdf.xacro (robot description, xacro)
@@ -1,67 +1,57 @@
 <?xml version="1.0"?>
-<robot xmlns:sensor="http://playerstage.sourceforge.net/gazebo/xmlschema/#sensor"
-xmlns:controller="http://playerstage.sourceforge.net/gazebo/xmlschema/#controller"
-xmlns:interface="http://playerstage.sourceforge.net/gazebo/xmlschema/#interface"
-xmlns:xacro="http://ros.org/wiki/xacro"
->
-  <!-- Quadrotor Sensor Plugins
-        <frameId>ardrone_base_link</frameId>
--->
-  <xacro:macro name="quadrotor_sensors">
-    <gazebo>
-      <plugin name="quadrotor_imu_sim" filename="libhector_gazebo_ros_imu.so">
-        <alwaysOn>true</alwaysOn>
-        <updateRate>100.0</updateRate>
-        <bodyName>base_link</bodyName>
-        <frameId>ardrone_base_link</frameId>
-        <topicName>/ardrone/imu</topicName>
-        <rpyOffsets>0 0 0</rpyOffsets> <!-- deprecated -->
-        <gaussianNoise>0</gaussianNoise>  <!-- deprecated -->
-        <accelDrift>0.5 0.5 0.5</accelDrift>
-        <accelGaussianNoise>0.35 0.35 0.3</accelGaussianNoise>
-        <rateDrift>0.0 0.0 0.0</rateDrift>
-        <rateGaussianNoise>0.00 0.00 0.00</rateGaussianNoise>
-        <headingDrift>0.0</headingDrift>
-        <headingGaussianNoise>0.00</headingGaussianNoise>
-      </plugin>
-      <plugin name="quadrotor_baro_sim" filename="libhector_gazebo_ros_baro.so">
-        <alwaysOn>true</alwaysOn>
-        <updateRate>10.0</updateRate>
-        <bodyName>base_link</bodyName>
-        <topicName>pressure_height</topicName>
-        <altimeterTopicName>altimeter</altimeterTopicName>
-        <offset>0</offset>
-        <drift>0.1</drift>
-        <gaussianNoise>0.5</gaussianNoise>
-      </plugin>
-      <plugin name="quadrotor_magnetic_sim" filename="libhector_gazebo_ros_magnetic.so">
-        <alwaysOn>true</alwaysOn>
-        <updateRate>10.0</updateRate>
-        <bodyName>base_link</bodyName>
-        <topicName>magnetic</topicName>
-        <offset>0 0 0</offset>
-        <drift>0.0 0.0 0.0</drift>
-        <gaussianNoise>1.3e-2 1.3e-2 1.3e-2</gaussianNoise>
-      </plugin>
-      <plugin name="quadrotor_gps_sim" filename="libhector_gazebo_ros_gps.so">
-        <alwaysOn>true</alwaysOn>
-        <updateRate>4.0</updateRate>
-        <bodyName>base_link</bodyName>
-        <topicName>fix</topicName>
-        <velocityTopicName>fix_velocity</velocityTopicName>
-        <drift>5.0 5.0 5.0</drift>
-        <gaussianNoise>0.1 0.1 0.1</gaussianNoise>
-        <velocityDrift>0 0 0</velocityDrift>
-        <velocityGaussianNoise>0.1 0.1 0.1</velocityGaussianNoise>
-      </plugin>
-      <plugin name="quadrotor_groundtruth_sim" filename="libgazebo_ros_p3d.so">
-        <alwaysOn>true</alwaysOn>
-        <updateRate>100.0</updateRate>
-        <bodyName>base_link</bodyName>
-        <topicName>ground_truth/state</topicName>
-        <gaussianNoise>0.0</gaussianNoise>
-        <frameName>map</frameName>
-      </plugin>
-    </gazebo>
-  </xacro:macro>
+<robot xmlns:xacro="http://ros.org/wiki/xacro">
+  <!-- Quadrotor Sensor Plugins -->
+  <gazebo>
+    <plugin name="quadrotor_imu_sim" filename="libhector_gazebo_ros_imu.so">
+      <updateRate>100.0</updateRate>
+      <bodyName>base_link</bodyName>
+      <frameId>ardrone_base_link</frameId>
+      <topicName>raw_imu</topicName>
+      <rpyOffsets>0 0 0</rpyOffsets> <!-- deprecated -->
+      <gaussianNoise>0</gaussianNoise>  <!-- deprecated -->
+      <accelDrift>0.5 0.5 0.5</accelDrift>
+      <accelGaussianNoise>0.35 0.35 0.3</accelGaussianNoise>
+      <rateDrift>0.1 0.1 0.1</rateDrift>
+      <rateGaussianNoise>0.05 0.05 0.015</rateGaussianNoise>
+    </plugin>
+    <plugin name="quadrotor_baro_sim" filename="libhector_gazebo_ros_baro.so">
+      <updateRate>10.0</updateRate>
+      <bodyName>base_link</bodyName>
+      <frameId>ardrone_base_link</frameId>
+      <topicName>pressure_height</topicName>
+      <altimeterTopicName>altimeter</altimeterTopicName>
+      <offset>0</offset>
+      <drift>10.0</drift>
+      <gaussianNoise>0.1</gaussianNoise>
+    </plugin>
+    <plugin name="quadrotor_magnetic_sim" filename="libhector_gazebo_ros_magnetic.so">
+      <updateRate>10.0</updateRate>
+      <bodyName>base_link</bodyName>
+      <frameId>ardrone_base_link</frameId>
+      <topicName>magnetic</topicName>
+      <offset>0 0 0</offset>
+      <drift>0.0 0.0 0.0</drift>
+      <gaussianNoise>1.3e-2 1.3e-2 1.3e-2</gaussianNoise>
+    </plugin>
+    <plugin name="quadrotor_gps_sim" filename="libhector_gazebo_ros_gps.so">
+      <updateRate>4.0</updateRate>
+      <bodyName>base_link</bodyName>
+      <frameId>ardrone_base_link</frameId>
+      <topicName>fix</topicName>
+      <velocityTopicName>fix_velocity</velocityTopicName>
+      <referenceLatitude>49.860246</referenceLatitude>
+      <referenceLongitude>8.687077</referenceLongitude>
+      <drift>5.0 5.0 5.0</drift>
+      <gaussianNoise>0.01 0.01 0.01</gaussianNoise>
+      <velocityDrift>0 0 0</velocityDrift>
+      <velocityGaussianNoise>0.05 0.05 0.05</velocityGaussianNoise>
+    </plugin>
+    <plugin name="quadrotor_groundtruth_sim" filename="libgazebo_ros_p3d.so">
+      <updateRate>100.0</updateRate>
+      <bodyName>base_link</bodyName>
+      <topicName>ground_truth/state</topicName>
+      <gaussianNoise>0.0</gaussianNoise>
+      <frameName>map</frameName>
+    </plugin>
+  </gazebo>
 </robot>
